Commit message: Added the imu links - visible on rviz

File: src/unitree_a2_mujoco/urdf/a2.urdf (robot description, URDF)
Before this commit: robot a2, 17 links, 16 joints
Links:
- added link imu_link, mass 0.0; collision sphere radius=0.01; visual sphere radius=0.01
Joints:
- added joint imu_joint: type fixed, parent base_link, child imu_link, origin xyz=0 0 0 rpy=0 0 0

Commit message: bridge to view lidar point clouds on rviz works. But the range finder sensors on mujoco are very glitchy

File: src/unitree_a2_mujoco/urdf/a2.urdf (robot description, URDF)
Before this commit: robot a2, 18 links, 17 joints
Links:
- added link lidar_link, mass 0.01; visual cylinder length=0.02 radius=0.02
Joints:
- added joint lidar_joint: type fixed, parent base_link, child lidar_link, origin xyz=0.3 0 0.15 rpy=0 0 -1.5708

Commit message: lidar works. The joint controllers are now  inactive in the launch file. This was done while testing if the lidar works.

File: src/unitree_a2_mujoco/urdf/a2.urdf (robot description, URDF)
Before this commit: robot a2, 19 links, 18 joints
Joints:
- joint lidar_joint: origin xyz=0.3 0 0.15 rpy=0 0 -1.5708 -> xyz=0 0 0.2 rpy=0 0 0
