Commit message: Lidar integrated

File: src/a2_description/urdf/a2.urdf (robot description, URDF)
Before this commit: robot a2, 18 links, 17 joints
Links:
- added link lidar_link, mass 0.001
Joints:
- added joint lidar_joint: type fixed, parent base_link, child lidar_link, origin xyz=0.0 0.0 0.2 rpy=0 0 0
